File: KiCAD/Display Adapters/Display Adapters.kicad_pcb (KiCad board)
At the start: 4 copper layers, 35.1 x 30.5 mm, 5 parts, among them J4 XT30PW_2_2_-M.G.B, J5 G46M2013201AWEU, J6 20455-040E-76

Commit message: guh
Parts:
- added H1: MountingHole_Pad, MountingHole:MountingHole_2.2mm_M2_DIN965_Pad_TopBottom, F.Cu at (164.2, 45.3)
- added H1: MountingHole_Pad, MountingHole:MountingHole_2.2mm_M2_DIN965_Pad_TopBottom, F.Cu at (77.5, 50.1)
- added H2: MountingHole_Pad, MountingHole:MountingHole_2.2mm_M2_DIN965_Pad_TopBottom, F.Cu at (133.5, 55.0)
- added H2: MountingHole_Pad, MountingHole:MountingHole_2.2mm_M2_DIN965_Pad_TopBottom, F.Cu at (103.3, 51.1)
- added J1: 20455-040E-76, SnapEDA:IPEX_20455-040E-76, F.Cu at (93.8, 42.5)
- added J2: G46M2013201AWEU, SnapEDA:AMPHENOL_G46M2013201AWEU, F.Cu at (95.1, 61.3)
- added J3: XT30PW_2_2_-M.G.B, SnapEDA:AMASS_XT30PW_2_2_-M.G.B, F.Cu at (80.9, 63.2)
Routing:
- net +5V: track 41.9 -> 106.5 mm, vias 1 -> 2
- net AUX_N: track 48.8 -> 104.5 mm, vias 1 -> 2
- net AUX_P: track 48.5 -> 104.1 mm, vias 1 -> 2
- net EDP_HPD: track 23.5 -> 68.3 mm
- net GND: track 16.3 -> 52.7 mm, vias 11 -> 40
- net 0_EDP_TX_N: track 20.5 -> 47.3 mm
- net 0_EDP_TX_P: track 20.5 -> 47.3 mm
- net 2_EDP_TX_N: track 21.5 -> 48.2 mm
- net 2_EDP_TX_P: track 21.5 -> 48.1 mm
- net BLK_PWM_LCD: track 24.0 -> 49.8 mm, vias 1 -> 2
- net 3_EDP_TX_P: track 20.6 -> 46.3 mm, vias 1 -> 2
- net 3_EDP_TX_N: track 20.6 -> 46.3 mm, vias 1 -> 2
- net BLK_OFF_N: track 29.5 -> 53.0 mm, vias 1 -> 2
- net 1_EDP_TX_N: track 20.8 -> 40.6 mm
- net 1_EDP_TX_P: track 20.8 -> 40.6 mm
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Other:
- board size 35.1 x 30.5 mm -> 97.3 x 31.8 mm
- board text added: "Source: EDP -> DP"
