File: KiCAD/Display Adapters/sink/sink.kicad_sch (KiCad schematic)
At the start: 5 parts, among them J4 XT30PW_2_2_-M.G.B, J5 G46M2013201AWEU, J6 20455-040E-76

Commit message: move into separate projects, fix wrong trace length on source
Parts:
- added H1, H2: MountingHole_Pad, MountingHole:MountingHole_2.2mm_M2_DIN965_Pad_TopBottom, symbol Mechanical:MountingHole_Pad
- renumbered C3 to C1, J4 to J1, J5 to J2, J6 to J3
Connections:
- net GND: now also H1.1, H2.1
Other:
- note added: "Mounting Holes"
- title: DP -> EDP -> (none)
- moved on the sheet: C1, C2, J1, J2, J3
