File: KiCAD/Display Adapters/sink/sink.kicad_pcb (KiCad board)
At the start: 4 copper layers, 38.2 x 36.4 mm, 7 parts, among them J1 47272-0001, J2 XT30PW_2_2_-M.G.B, J3 20455-040E-76

Commit message: updates
Parts:
- moved C2 13.2 mm to (165.4, 100.0), turned to 90 degrees
- moved C1 7.58 mm to (171.6, 99.9), turned to -90 degrees
- moved J3 2.89 mm to (171.1, 94.5), turned to 180 degrees
- moved J2 2.59 mm to (158.9, 121.9)
Connections:
- J1 pad 1: 0_EDP_TX_P -> 3_EDP_TX_N
- J1 pad 10: 3_EDP_TX_P -> 0_EDP_TX_N
- J1 pad 12: 3_EDP_TX_N -> 0_EDP_TX_P
- J1 pad 3: 0_EDP_TX_N -> 3_EDP_TX_P
- J1 pad 4: 1_EDP_TX_P -> 2_EDP_TX_N
- J1 pad 6: 1_EDP_TX_N -> 2_EDP_TX_P
- J1 pad 7: 2_EDP_TX_P -> 1_EDP_TX_N
- J1 pad 9: 2_EDP_TX_N -> 1_EDP_TX_P
Routing:
- net AUX_N: track 47.9 -> 18.1 mm
- net AUX_P: track 47.8 -> 18.1 mm
- net +5V: track 48.6 -> 23.1 mm
- net 0_EDP_TX_P: track 31.2 -> 18.5 mm
- net 0_EDP_TX_N: track 31.2 -> 18.5 mm
- net 1_EDP_TX_P: track 31.2 -> 18.5 mm
- net 1_EDP_TX_N: track 31.2 -> 18.5 mm
- net 2_EDP_TX_P: track 31.1 -> 18.5 mm
- net 3_EDP_TX_P: track 31.1 -> 18.5 mm
- net 3_EDP_TX_N: track 31.1 -> 18.5 mm
- net 2_EDP_TX_N: track 31.1 -> 18.5 mm
- net BLK_OFF_N: track 35.4 -> 23.9 mm
- net BLK_PWM_LCD: track 25.2 -> 20.0 mm
- net GND: track 24.7 -> 27.5 mm
- net EDP_HPD: track 20.2 -> 21.9 mm, vias 2 -> 0
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Other:
- board size 38.2 x 36.4 mm -> 40.4 x 36.4 mm
- board text added: "JLCJLCJLCJLC"
- board text added: "Sink: DP -> EDP"
- board text added: "chinh4"
