File: KiCAD/Display Adapters/source/source.kicad_sch (KiCad schematic)
At the start: 5 parts, among them J1 20455-040E-76, J2 G46M2013201AWEU, J3 XT30PW_2_2_-M.G.B

Commit message: move into separate projects, fix wrong trace length on source
Parts:
- renumbered J3 to J2, J2 to J3
Other:
- title: EDP -> DP -> (none)
- moved on the sheet: H1, H2, J1, J2, J3
