File: KiCAD/Display Adapters/source/source.kicad_pcb (KiCad board)
At the start: 4 copper layers, 40 x 30.3 mm, 5 parts, among them J1 20455-040E-76, J2 47272-0001, J3 XT30PW_2_2_-M.G.B

Commit message: updates
Parts:
- moved J1 1.35 mm to (131.8, 57.9)
Routing:
- net AUX_P: track 33.3 -> 35.0 mm
- net AUX_N: track 33.3 -> 35.0 mm
- net GND: track 26.8 -> 27.8 mm, vias 19 -> 20
- net EDP_HPD: track 24.3 -> 25.0 mm
- net BLK_PWM_LCD: track 32.7 -> 32.2 mm
