File: KiCAD/Keyboard/frameortho.kicad_pcb (KiCad board)
At the start: 2 copper layers, 226 x 105 mm, 142 parts, among them SW1 SW_Push, SW2 SW_Push, U1 RP2040, U2 W25Q128JVS, U3 XC6206PxxxMR, Y1 12 MHz 18pF

Commit message: add ground vias around usb vias
Routing:
- net GND: track 101.7 -> 90.1 mm, vias 39 -> 42
Changed lines of the file:
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@@
-	)
-	(segment
-		(start 208.6102 106.7816)
-		(end 208.3562 106.5276)
-		(width 0.3048)
-		(layer "F.Cu")
-		(net 59)
 	)
 	(segment
@@
 	)
 	(segment
-		(start 208.3562 106.5276)
-		(end 204.3456 106.5276)
-		(width 0.3048)
-		(layer "F.Cu")
-		(net 59)
-	)
-	(segment
 		(start 216.9388 110.2614)
 		(end 217.1192 110.2614)
@@
 	)
 	(segment
+		(start 208.6102 106.5202)
+		(end 208.61 106.52)
+		(width 0.3048)
+		(layer "F.Cu")
+		(net 59)
+	)
+	(segment
 		(start 212.3186 100.2538)
 		(end 211.9376 99.8728)
@@
 		(start 221.107 108.8644)
 		(end 221.3356 109.093)
-		(width 0.3048)
-		(layer "F.Cu")
-		(net 59)
-	)
-	(segment
-		(start 204.3456 106.5276)
-		(end 203.8376 106.0196)
 		(width 0.3048)
 		(layer "F.Cu")
@@
 	)
 	(segment
-		(start 208.6102 108.4387)
-		(end 208.6102 106.7816)
-		(width 0.3048)
-		(layer "F.Cu")
-		(net 59)
-	)
-	(segment
 		(start 215.766067 106.636133)
 		(end 216.281 106.1212)
@@
 	)
 	(segment
+		(start 208.6102 108.4387)
+		(end 208.6102 106.5202)
+		(width 0.3048)
+		(layer "F.Cu")
+		(net 59)
+	)
+	(segment
 		(start 215.773867 107.4446)
 		(end 215.766067 107.4524)
@@
 	)
 	(segment
-		(start 203.8376 106.0196)
-		(end 203.8376 99.2632)
-		(width 0.3048)
-		(layer "F.Cu")
-		(net 59)
-	)
-	(segment
 		(start 222.0568 123.2562)
 		(end 223.0374 122.2756)
@@
 	)
 	(via
+		(at 210.861602 90.043)
+		(size 0.6)
+		(drill 0.3)
+		(layers "F.Cu" "B.Cu")
+		(free yes)
+		(net 59)
+	)
+	(via
 		(at 213.23654 113.9435)
 		(size 0.6)
@@
 		(size 0.6)
 		(drill 0.3)
+		(layers "F.Cu" "B.Cu")
+		(net 59)
+	)
+	(via
+		(at 213.711602 90.043)
+		(size 0.6)
+		(drill 0.3)
+		(layers "F.Cu" "B.Cu")
+		(free yes)
+		(net 59)
+	)
+	(via
+		(at 208.61 106.52)
+		(size 0.6)
+		(drill 0.3)

Commit message: fix schematics
Parts:
- renumbered TP24 to 1.1V, TP23 to 3.3V, TP25 to GND
Routing:
- net GND: track 90.1 -> 61.1 mm
