File: KiCAD/Keyboard/frameortho.kicad_pcb (KiCad board)
At the start: 2 copper layers, 226 x 105 mm, 142 parts, among them SW1 SW_Push, SW2 SW_Push, U1 RP2040, U2 W25Q128JVS, U3 XC6206PxxxMR, Y1 12 MHz 18pF

Commit message: label
Other:
- board text added: "chinh4"
- board text added: "frameortho"
Changed lines of the file:
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@@
+		)
+	)
+	(gr_text "frameortho"
+		(at 205.793683 182.82 0)
+		(layer "F.SilkS")
+		(effects
+			(font
+				(size 1.5 1.5)
+				(thickness 0.3)
+				(bold yes)
+			)
+			(justify left bottom)
 		)
 	)
@@
 		)
 	)
+	(gr_text "chinh4"
+		(at 325.27 184.82 -0)
+		(layer "B.SilkS")
+		(effects
+			(font
+				(size 1.5 1.5)
+				(thickness 0.3)
+				(bold yes)
+			)
+			(justify left bottom mirror)
+		)
+	)
