File: KiCAD/USB/usb-hub.kicad_sch (KiCad schematic)
At the start: 22 parts, among them J1 046809610110846+ Male, J2 046809610110846+ Female, J3 Conn_01x04_Socket, U1 CY7C65634-28LTXC, Y1 12MHz 18pF

Commit message: fix schematics
Parts:
- C10, C9: value 33 pF -> 27 pF
Changed lines of the file:
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@@
 			)
 		)
-		(property "Value" "33 pF"
+		(property "Value" "27 pF"
 			(at 81.2863 134.62 0)
 			(effects
@@
 			)
 		)
-		(property "Value" "33 pF"
+		(property "Value" "27 pF"
 			(at 104.394 134.62 0)
 			(effects
