File: KiCAD/USB (v2)/usb-hub.kicad_pcb (KiCad board)
At the start: 2 copper layers, 22.4 x 24.2 mm, 22 parts, among them J1 046809610110846+ Male, J3 Conn_01x04_Socket, U1 CY7C65634-28LTXC, Y1 12MHz 18pF

Commit message: label
Routing:
- net USB_HOST_P: track 24.0 -> 19.7 mm
- net USB_HOST_N: track 23.9 -> 20.1 mm
- net GND: vias 26 -> 30
